Commit message: Updating urdf and model 3

File: src/Universal_Robots_ROS2_Tutorials/my_dual_robot_cell/my_dual_robot_cell_description/urdf/my_dual_robot_cell.urdf.xacro (robot description, xacro)
@@ -27,5 +27,5 @@
     bob_visual_parameters_file="$(arg bob_visual_parameters_file)"
     >
-      <origin xyz="0 0 1" rpy="0 0 0" />
+      <origin xyz="0 0 0" rpy="0 0 0" />
   </xacro:my_dual_robot_cell>
 </robot>
