Commit message: added mir to rviz

File: src/Universal_Robots_ROS2_Tutorials/my_dual_robot_cell/my_dual_robot_cell_description/urdf/my_dual_robot_cell_macro.xacro (robot description, xacro)
@@ -16,72 +16,38 @@
     bob_visual_parameters_file
     ">
-    <joint name="table_base_joint" type="fixed">
+    <joint name="mir_base_joint" type="fixed">
       <xacro:insert_block name="origin" />
       <parent link="${parent}" />
-      <child link="table" />
+      <child link="mir" />
     </joint>
-    <link name="table">
+    <link name="mir">
       <visual>
         <geometry>
-          <mesh filename="package://my_robot_cell_description/meshes/fzi_table.dae"/>
+          <mesh filename="package://my_robot_cell_description/meshes/Dual_Robot_Base.dae"/>
         </geometry>
-        <origin rpy="0 0 0" xyz="0.75 0.5 -1"/>
+        <origin rpy="1.570796 0 0" xyz="0 0 -0.70"/>
       </visual>
       <collision>
         <geometry>
-          <mesh filename="package://my_robot_cell_description/meshes/fzi_table.dae"/>
+          <mesh filename="package://my_robot_cell_description/meshes/Dual_Robot_Base.dae"/>
         </geometry>
-        <origin rpy="0 0 0" xyz="0.75 0.5 -1"/>
+        <origin rpy="1.570796 0 0" xyz="0 0 -0.70"/>
       </collision>
     </link>
-    <link name="monitor">
-      <visual>
-        <geometry>
-          <mesh filename="package://my_robot_cell_description/meshes/171005_Motek_Monitor_L.dae"/>
-        </geometry>
-      </visual>
-      <collision>
-        <geometry>
-          <mesh filename="package://my_robot_cell_description/meshes/171005_Motek_Monitor_L.dae"/>
-        </geometry>
-      </collision>
-    </link>
-    <joint name="base_to_monitor" type="fixed">
-      <parent link="table"/>
-      <child link="monitor"/>
-      <origin xyz="0.2 0.6 0"/>
-    </joint>
     <material name="white">
       <color rgba="1 1 1 1"/>
     </material>
-    <link name="wall">
-      <visual>
-        <geometry>
-          <mesh filename="package://my_robot_cell_description/meshes/wall.dae"/>
-        </geometry>
-      </visual>
-      <collision>
-        <geometry>
-          <box size="4.44 0.1 2.5"/>
-        </geometry>
-      </collision>
-    </link>
-    <joint name="base_to_wall" type="fixed">
-      <parent link="table"/>
-      <child link="wall"/>
-      <origin xyz="1.25 1.5 0.5"/>
-    </joint>
     <!--Creates the mounts to attach the robots to the table-->
     <link name="alice_robot_mount"/>
     <joint name="base_to_alice_robot_mount" type="fixed">
-      <parent link="table"/>
+      <parent link="mir"/>
       <child link="alice_robot_mount"/>
-      <origin xyz="0.5 0.3 0" rpy="0 0 ${pi}" />
+      <origin xyz="0 -0.33 -0.3" rpy="0 0 ${pi}" />
     </joint>
     <link name="bob_robot_mount"/>
     <joint name="base_to_bob_robot_mount" type="fixed">
-      <parent link="table"/>
+      <parent link="mir"/>
       <child link="bob_robot_mount"/>
-      <origin xyz="1.2 0.3 0" rpy="0 0 ${pi}" />
+      <origin xyz="0 0.33 -0.3" rpy="0 0 ${pi}" />
     </joint>
     <!--Creates the 1st Robot-->

Commit message: made the mir low res

File: src/Universal_Robots_ROS2_Tutorials/my_dual_robot_cell/my_dual_robot_cell_description/urdf/my_dual_robot_cell_macro.xacro (robot description, xacro)
@@ -21,16 +21,30 @@
       <child link="mir" />
     </joint>
+	<!--<link name="mir">-->
+	<!--<visual>-->
+	<!--<geometry>-->
+	<!--<mesh filename="package://my_robot_cell_description/meshes/High_Res_Dual_Robot_Base.dae"/>-->
+	<!--</geometry>-->
+	<!--<origin rpy="1.570796 0 0" xyz="0 0 -0.70"/>-->
+	<!--</visual>-->
+	<!--<collision>-->
+	<!--<geometry>-->
+	<!--<mesh filename="package://my_robot_cell_description/meshes/High_Res_Dual_Robot_Base.dae"/>-->
+	<!--</geometry>-->
+	<!--<origin rpy="1.570796 0 0" xyz="0 0 -0.70"/>-->
+	<!--</collision>-->
+	<!--</link>-->
     <link name="mir">
       <visual>
         <geometry>
-          <mesh filename="package://my_robot_cell_description/meshes/Dual_Robot_Base.dae"/>
+          <mesh filename="package://my_robot_cell_description/meshes/Low_Res_Dual_Robot_Base.dae"/>
         </geometry>
-        <origin rpy="1.570796 0 0" xyz="0 0 -0.70"/>
+        <origin rpy="1.570796 0 1.570796" xyz="0.26 -0.4 -1.0"/>
       </visual>
       <collision>
         <geometry>
-          <mesh filename="package://my_robot_cell_description/meshes/Dual_Robot_Base.dae"/>
+          <mesh filename="package://my_robot_cell_description/meshes/Low_Res_Dual_Robot_Base.dae"/>
         </geometry>
-        <origin rpy="1.570796 0 0" xyz="0 0 -0.70"/>
+        <origin rpy="1.570796 0 1.570796" xyz="0.26 -0.4 -1.0"/>
       </collision>
     </link>

Commit message: WIP on main

File: src/Universal_Robots_ROS2_Tutorials/my_dual_robot_cell/my_dual_robot_cell_description/urdf/my_dual_robot_cell_macro.xacro (robot description, xacro)
@@ -21,30 +21,16 @@
       <child link="mir" />
     </joint>
-	<!--<link name="mir">-->
-	<!--<visual>-->
-	<!--<geometry>-->
-	<!--<mesh filename="package://my_robot_cell_description/meshes/High_Res_Dual_Robot_Base.dae"/>-->
-	<!--</geometry>-->
-	<!--<origin rpy="1.570796 0 0" xyz="0 0 -0.70"/>-->
-	<!--</visual>-->
-	<!--<collision>-->
-	<!--<geometry>-->
-	<!--<mesh filename="package://my_robot_cell_description/meshes/High_Res_Dual_Robot_Base.dae"/>-->
-	<!--</geometry>-->
-	<!--<origin rpy="1.570796 0 0" xyz="0 0 -0.70"/>-->
-	<!--</collision>-->
-	<!--</link>-->
     <link name="mir">
       <visual>
         <geometry>
-          <mesh filename="package://my_robot_cell_description/meshes/Low_Res_Dual_Robot_Base.dae"/>
+          <mesh filename="package://my_robot_cell_description/meshes/Dual_Robot_Base.dae"/>
         </geometry>
-        <origin rpy="1.570796 0 1.570796" xyz="0.26 -0.4 -1.0"/>
+        <origin rpy="1.570796 0 0" xyz="0 0 -0.70"/>
       </visual>
       <collision>
         <geometry>
-          <mesh filename="package://my_robot_cell_description/meshes/Low_Res_Dual_Robot_Base.dae"/>
+          <mesh filename="package://my_robot_cell_description/meshes/Dual_Robot_Base.dae"/>
         </geometry>
-        <origin rpy="1.570796 0 1.570796" xyz="0.26 -0.4 -1.0"/>
+        <origin rpy="1.570796 0 0" xyz="0 0 -0.70"/>
       </collision>
     </link>

Commit message: added a launch scrip for the sim

File: src/Universal_Robots_ROS2_Tutorials/my_dual_robot_cell/my_dual_robot_cell_description/urdf/my_dual_robot_cell_macro.xacro (robot description, xacro)
@@ -52,4 +52,23 @@
       <color rgba="1 1 1 1"/>
     </material>
+    <joint name="table" type="fixed">
+      <xacro:insert_block name="origin" />
+      <parent link="world" />
+      <child link="table" />
+    </joint>
+    <link name="table">
+      <visual>
+        <geometry>
+          <mesh filename="package://my_robot_cell_description/meshes/fzi_table.dae"/>
+        </geometry>
+        <origin rpy="0 0 0" xyz="0.75 0.5 -1"/>
+      </visual>
+      <collision>
+        <geometry>
+          <mesh filename="package://my_robot_cell_description/meshes/fzi_table.dae"/>
+        </geometry>
+        <origin rpy="0 0 0" xyz="0.75 0.5 -1"/>
+      </collision>
+    </link>
     <!--Creates the mounts to attach the robots to the table-->
     <link name="alice_robot_mount"/>

Commit message: updated low res base

File: src/Universal_Robots_ROS2_Tutorials/my_dual_robot_cell/my_dual_robot_cell_description/urdf/my_dual_robot_cell_macro.xacro (robot description, xacro)
@@ -21,16 +21,30 @@
       <child link="mir" />
     </joint>
+	<!--<link name="mir">-->
+	<!--<visual>-->
+	<!--<geometry>-->
+	<!--<mesh filename="package://my_robot_cell_description/meshes/Dual_Robot_Base.dae"/>-->
+	<!--</geometry>-->
+	<!--<origin rpy="1.570796 0 0" xyz="0 0 -0.70"/>-->
+	<!--</visual>-->
+	<!--<collision>-->
+	<!--<geometry>-->
+	<!--<mesh filename="package://my_robot_cell_description/meshes/Dual_Robot_Base.dae"/>-->
+	<!--</geometry>-->
+	<!--<origin rpy="1.570796 0 0" xyz="0 0 -0.70"/>-->
+	<!--</collision>-->
+	<!--</link>-->
     <link name="mir">
       <visual>
         <geometry>
-          <mesh filename="package://my_robot_cell_description/meshes/Dual_Robot_Base.dae"/>
+          <mesh filename="package://my_robot_cell_description/meshes/Low_Res_Dual_Robot_Base.dae"/>
         </geometry>
-        <origin rpy="1.570796 0 0" xyz="0 0 -0.70"/>
+        <origin rpy="1.570796 0 1.570796" xyz="0.25 -0.4 -1.0"/>
       </visual>
       <collision>
         <geometry>
-          <mesh filename="package://my_robot_cell_description/meshes/Dual_Robot_Base.dae"/>
+          <mesh filename="package://my_robot_cell_description/meshes/Low_Res_Dual_Robot_Base.dae"/>
         </geometry>
-        <origin rpy="1.570796 0 0" xyz="0 0 -0.70"/>
+		<origin rpy="1.570796 0 1.570796" xyz="0.25 -0.4 -1.0"/>
       </collision>
     </link>

Commit message: removed table so bob can run servo

File: src/Universal_Robots_ROS2_Tutorials/my_dual_robot_cell/my_dual_robot_cell_description/urdf/my_dual_robot_cell_macro.xacro (robot description, xacro)
@@ -52,23 +52,23 @@
       <color rgba="1 1 1 1"/>
     </material>
-    <joint name="table" type="fixed">
-      <xacro:insert_block name="origin" />
-      <parent link="world" />
-      <child link="table" />
-    </joint>
-    <link name="table">
-      <visual>
-        <geometry>
-          <mesh filename="package://my_robot_cell_description/meshes/fzi_table.dae"/>
-        </geometry>
-        <origin rpy="0 0 0" xyz="0.75 0.5 -1"/>
-      </visual>
-      <collision>
-        <geometry>
-          <mesh filename="package://my_robot_cell_description/meshes/fzi_table.dae"/>
-        </geometry>
-        <origin rpy="0 0 0" xyz="0.75 0.5 -1"/>
-      </collision>
-    </link>
+	<!--<joint name="table" type="fixed">-->
+	<!--<xacro:insert_block name="origin" />-->
+	<!--<parent link="world" />-->
+	<!--<child link="table" />-->
+	<!--</joint>-->
+	<!--<link name="table">-->
+	<!--<visual>-->
+	<!--<geometry>-->
+	<!--<mesh filename="package://my_robot_cell_description/meshes/fzi_table.dae"/>-->
+	<!--</geometry>-->
+	<!--<origin rpy="0 0 0" xyz="0.75 0.5 -1"/>-->
+	<!--</visual>-->
+	<!--<collision>-->
+	<!--<geometry>-->
+	<!--<mesh filename="package://my_robot_cell_description/meshes/fzi_table.dae"/>-->
+	<!--</geometry>-->
+	<!--<origin rpy="0 0 0" xyz="0.75 0.5 -1"/>-->
+	<!--</collision>-->
+	<!--</link>-->
     <!--Creates the mounts to attach the robots to the table-->
     <link name="alice_robot_mount"/>

Commit message: added admittance and gripping function in executer, and updated admittance control so it publish to same frame as it gets in

File: src/Universal_Robots_ROS2_Tutorials/my_dual_robot_cell/my_dual_robot_cell_description/urdf/my_dual_robot_cell_macro.xacro (robot description, xacro)
@@ -40,5 +40,5 @@
           <mesh filename="package://my_robot_cell_description/meshes/Low_Res_Dual_Robot_Base.dae"/>
         </geometry>
-        <origin rpy="1.570796 0 1.570796" xyz="0.25 -0.4 -1.0"/>
+        <origin rpy="1.570796 0 1.570796" xyz="-0.25 -0.1 -0.2"/>
       </visual>
       <collision>
@@ -46,5 +46,5 @@
           <mesh filename="package://my_robot_cell_description/meshes/Low_Res_Dual_Robot_Base.dae"/>
         </geometry>
-		<origin rpy="1.570796 0 1.570796" xyz="0.25 -0.4 -1.0"/>
+		<origin rpy="1.570796 0 1.570796" xyz="-0.25 -0.1 -0.2"/>
       </collision>
     </link>
@@ -76,5 +76,5 @@
       <parent link="mir"/>
       <child link="alice_robot_mount"/>
-      <origin xyz="0 -0.33 -0.3" rpy="0 0 ${pi}" />
+	  <origin xyz="0 -0.33 -0.3" rpy="${-pi/4} 0 ${pi}" />
     </joint>
     <link name="bob_robot_mount"/>
@@ -82,5 +82,5 @@
       <parent link="mir"/>
       <child link="bob_robot_mount"/>
-      <origin xyz="0 0.33 -0.3" rpy="0 0 ${pi}" />
+	  <origin xyz="0 0.33 -0.3" rpy="${pi/4} 0 ${pi}" />
     </joint>
     <!--Creates the 1st Robot-->

Commit message: Updating urdf and model

File: src/Universal_Robots_ROS2_Tutorials/my_dual_robot_cell/my_dual_robot_cell_description/urdf/my_dual_robot_cell_macro.xacro (robot description, xacro)
@@ -40,5 +40,5 @@
           <mesh filename="package://my_robot_cell_description/meshes/Low_Res_Dual_Robot_Base.dae"/>
         </geometry>
-        <origin rpy="1.570796 0 1.570796" xyz="-0.25 -0.1 -0.2"/>
+        <origin rpy="1.570796 0 1.570796" xyz="0.0 0.0 0.0"/>
       </visual>
       <collision>
@@ -46,5 +46,5 @@
           <mesh filename="package://my_robot_cell_description/meshes/Low_Res_Dual_Robot_Base.dae"/>
         </geometry>
-		<origin rpy="1.570796 0 1.570796" xyz="-0.25 -0.1 -0.2"/>
+		<origin rpy="1.570796 0 1.570796" xyz="0.0 0.0 0.0"/>
       </collision>
     </link>

Commit message: Updating urdf and model 2

File: src/Universal_Robots_ROS2_Tutorials/my_dual_robot_cell/my_dual_robot_cell_description/urdf/my_dual_robot_cell_macro.xacro (robot description, xacro)
@@ -40,5 +40,5 @@
           <mesh filename="package://my_robot_cell_description/meshes/Low_Res_Dual_Robot_Base.dae"/>
         </geometry>
-        <origin rpy="1.570796 0 1.570796" xyz="0.0 0.0 0.0"/>
+        <origin rpy="0.0 0.0 0.0" xyz="0.0 0.0 0.0"/>
       </visual>
       <collision>
@@ -46,5 +46,5 @@
           <mesh filename="package://my_robot_cell_description/meshes/Low_Res_Dual_Robot_Base.dae"/>
         </geometry>
-		<origin rpy="1.570796 0 1.570796" xyz="0.0 0.0 0.0"/>
+		<origin rpy="0.0 0.0 0.0" xyz="0.0 0.0 0.0"/>
       </collision>
     </link>

Commit message: new urdf for bob and alice

File: src/Universal_Robots_ROS2_Tutorials/my_dual_robot_cell/my_dual_robot_cell_description/urdf/my_dual_robot_cell_macro.xacro (robot description, xacro)
@@ -76,5 +76,5 @@
       <parent link="mir"/>
       <child link="alice_robot_mount"/>
-	  <origin xyz="0 -0.33 -0.3" rpy="${-pi/4} 0 ${pi}" />
+	  <origin xyz="-0.2339 0.0083 0.7755" rpy="-0.6319 0.5207 2.1817" />
     </joint>
     <link name="bob_robot_mount"/>
@@ -82,5 +82,5 @@
       <parent link="mir"/>
       <child link="bob_robot_mount"/>
-	  <origin xyz="0 0.33 -0.3" rpy="${pi/4} 0 ${pi}" />
+	  <origin xyz="0.1919 0.0040 0.7850" rpy="-0.5832 0.5376 -0.9286" />
     </joint>
     <!--Creates the 1st Robot-->
